File: diodeplate.kicad_sch (KiCad schematic)
At the start: 86 parts, among them U1 TS-1185EC-C-D-B, U10 CP2102-GMR, U11 U262-16XN-4BVC11, U14 UMH3N, U2 TS-1185EC-C-D-B, U3 TS-1185EC-C-D-B, U8 ESP32-WROOM-32E(4MB), U9 SN74AHCT32QPWRQ1

Commit message: add first pcb design
Parts:
- removed C13: 10uF, Capacitor_SMD:C_0603_1608Metric_Pad1.08x0.95mm_HandSolder, symbol Device:C
- removed F1: BSMD1812-300-16V, footprint:F1812, symbol lcsc:BSMD1812-300-16V
- removed LED1, LED10, LED11, LED12, LED13, LED14, LED15, LED16, LED17, LED18, LED19, LED2, LED20, LED21, LED22, LED23, LED24, LED25, LED26, LED27, LED28, LED29, LED3, LED30, LED4, LED5, LED6, LED7, LED8, LED9: XL-5050RGBC-WS2812B, footprint:LED-SMD_4P-L5.0-W5.0-BL_XL-5050RGBC, symbol lcsc:XL-5050RGBC-WS2812B
- removed REF1: BL1117-33CX, footprint:SOT-223-4_L6.5-W3.5-P2.30-LS7.0-BR, symbol lcsc:BL1117-33CX
- removed U1, U2, U3: TS-1185EC-C-D-B, footprint:SW-SMD_4P-L3.7-W3.0-P1.50-LS4.7, symbol lcsc:TS-1185EC-C-D-B
- removed U10: CP2102-GMR, footprint:QFN-28_L5.0-W5.0-P0.50-BL-EP, symbol lcsc:CP2102-GMR
- removed U11: U262-16XN-4BVC11, footprint:USB-3.1-SMD_U262-161N-4BVC11, symbol lcsc:U262-16XN-4BVC11
- removed U14: UMH3N, footprint:SC-70-6_L2.2-W1.3-P0.65-LS2.1-BR, symbol lcsc:UMH3N
- removed U8: ESP32-WROOM-32E(4MB), footprint:WIFI-SMD_ESP32-WROOM-32E, symbol lcsc:ESP32-WROOM-32E(4MB)
- removed U9: SN74AHCT32QPWRQ1, footprint:TSSOP-14_L5.0-W4.4-P0.65-LS6.5-BL, symbol lcsc:SN74AHCT32QPWRQ1
- added F1: BSMD1812-300-16V, footprint:F1812, symbol GLOWINGKITTYPARTS:BSMD1812-300-16V
- added LED1, LED10, LED11, LED12, LED13, LED14, LED15, LED16, LED17, LED18, LED19, LED2, LED20, LED21, LED22, LED23, LED24, LED25, LED26, LED27, LED28, LED29, LED3, LED30, LED4, LED5, LED6, LED7, LED8, LED9: XL-5050RGBC-WS2812B, footprint:LED-SMD_4P-L5.0-W5.0-BL_XL-5050RGBC, symbol GLOWINGKITTYPARTS:XL-5050RGBC-WS2812B
- added SW1, SW2, SW3: TS-1185EC-C-D-B, footprint:SW-SMD_4P-L3.7-W3.0-P1.50-LS4.7, symbol GLOWINGKITTYPARTS:TS-1185EC-C-D-B
- added U1: ESP32-WROOM-32E, footprint:WIFI-SMD_ESP32-WROOM-32E, symbol GLOWINGKITTYPARTS:ESP32-WROOM-32E
- added U2: CP2102-GMR, footprint:QFN-28_L5.0-W5.0-P0.50-BL-EP, symbol GLOWINGKITTYPARTS:CP2102-GMR
- added U3: U262-161N-4BVC11, footprint:USB-3.1-SMD_U262-161N-4BVC11, symbol GLOWINGKITTYPARTS:U262-161N-4BVC11
- added U4: BL1117-33CX, footprint:SOT-223-4_L6.5-W3.5-P2.30-LS7.0-BR, symbol GLOWINGKITTYPARTS:BL1117-33CX
- added U5: UMH3N, footprint:SC-70-6_L2.2-W1.3-P0.65-LS2.1-BR, symbol GLOWINGKITTYPARTS:UMH3N
- added U6: SN74AHCT32QPWRQ1, footprint:TSSOP-14_L5.0-W4.4-P0.65-LS6.5-BL, symbol GLOWINGKITTYPARTS:SN74AHCT32QPWRQ1
Connections:
- net +3V3: now also C1.1, U1.2 (3V3), U2.6 (VDD), U2.7 (REGIN), U4.2 (Vout), U4.4 (Vout); no longer C1.2
- net +5V: now also F1.2, LED1.1 (VDD), LED10.1 (VDD), LED11.1 (VDD), LED12.1 (VDD), LED13.1 (VDD), LED14.1 (VDD), LED15.1 (VDD), LED16.1 (VDD), LED17.1 (VDD), LED18.1 (VDD), LED19.1 (VDD), LED2.1 (VDD), LED20.1 (VDD), LED21.1 (VDD), LED22.1 (VDD), LED23.1 (VDD), LED24.1 (VDD), LED25.1 (VDD), LED26.1 (VDD), LED27.1 (VDD), LED28.1 (VDD), LED29.1 (VDD), LED3.1 (VDD), LED30.1 (VDD), LED4.1 (VDD), LED5.1 (VDD), LED6.1 (VDD), LED7.1 (VDD), LED8.1 (VDD), LED9.1 (VDD), U2.8 (VBUS), U4.3 (Vin), U6.14 (VCC)
- net DTR: now also U2.28 (DTR), U5.2 (B), U5.4 (E)
- net GND: now also C1.2, LED1.4 (GND), LED10.4 (GND), LED11.4 (GND), LED12.4 (GND), LED13.4 (GND), LED14.4 (GND), LED15.4 (GND), LED16.4 (GND), LED17.4 (GND), LED18.4 (GND), LED19.4 (GND), LED2.4 (GND), LED20.4 (GND), LED21.4 (GND), LED22.4 (GND), LED23.4 (GND), LED24.4 (GND), LED25.4 (GND), LED26.4 (GND), LED27.4 (GND), LED28.4 (GND), LED29.4 (GND), LED3.4 (GND), LED30.4 (GND), LED4.4 (GND), LED5.4 (GND), LED6.4 (GND), LED7.4 (GND), LED8.4 (GND), LED9.4 (GND), SW1.1, SW2.1, SW3.1, U1.1 (GND), U1.15 (GND), U1.38 (GND), U1.39 (GND), U2.3 (GND), U3.A1B12 (GND), U3.B1A12 (GND), U3.SHELL, U4.1 (GND), U6.10 (3B), U6.11 (4Y), U6.12 (4A), U6.13 (4B), U6.2 (1B), U6.4 (2A), U6.5 (2B), U6.6 (2Y), U6.7 (GND), U6.8 (3Y), U6.9 (3A); no longer C1.1
- net IO0: now also U1.25 (IO0), U5.3 (C)
- net IO16/LED1: now also U1.27 (IO16), U6.1 (1A)
- net IO33/MAINBUTTON: now also SW3.2, U1.9 (IO33)
- net LED DATA OUT: now also LED1.3 (DI)
- net RESET: now also U1.3 (EN), U5.6 (C)
- net RTS: now also U2.27 (DSR), U5.1 (E), U5.5 (B)
- net RXD: now also U1.34 (RXD0), U2.26 (TXD)
- net TXD: now also U1.35 (TXD0), U2.25 (RXD)
- net USB-C CC1: now also U3.A5 (CC1)
- net USB-C CC2: now also U3.B5 (CC2)
- net USB-C DATA +: now also U2.4 (D+), U3.A6 (DP1), U3.B6 (DP2)
- net USB-C DATA -: now also U2.5 (D-), U3.A7 (DN1), U3.B7 (DN2)
- net VBUS: now also F1.1, U3.A4B9 (VBUS), U3.B4A9 (VBUS)
- net at R4.1: now also SW1.2
- net at R5.1: now also SW2.2
- net at R1.2: now also U6.3 (1Y)
- new net: LED2.2 (DO), LED3.3 (DI)
- new net: LED1.2 (DO), LED2.3 (DI)
- new net: LED25.2 (DO), LED26.3 (DI)
- new net: LED24.2 (DO), LED25.3 (DI)
- new net: LED5.2 (DO), LED6.3 (DI)
- new net: LED4.2 (DO), LED5.3 (DI)
- new net: LED7.2 (DO), LED8.3 (DI)
- new net: LED6.2 (DO), LED7.3 (DI)
- new net: LED16.2 (DO), LED17.3 (DI)
- new net: LED15.2 (DO), LED16.3 (DI)
- new net: LED17.2 (DO), LED18.3 (DI)
- new net: LED3.2 (DO), LED4.3 (DI)
- new net: LED8.2 (DO), LED9.3 (DI)
- new net: LED21.2 (DO), LED22.3 (DI)
- new net: LED20.2 (DO), LED21.3 (DI)
- new net: LED27.2 (DO), LED28.3 (DI)
- new net: LED26.2 (DO), LED27.3 (DI)
- new net: LED10.2 (DO), LED11.3 (DI)
- new net: LED10.3 (DI), LED9.2 (DO)
- new net: LED29.2 (DO), LED30.3 (DI)
- new net: LED18.2 (DO), LED19.3 (DI)
- new net: LED28.2 (DO), LED29.3 (DI)
- new net: LED14.2 (DO), LED15.3 (DI)
- new net: LED13.2 (DO), LED14.3 (DI)
- new net: LED12.2 (DO), LED13.3 (DI)
- new net: U1.17 (NC), U1.18 (NC), U1.19 (NC), U1.20 (NC), U1.21 (NC), U1.22 (NC)
- new net: LED11.2 (DO), LED12.3 (DI)
- new net: LED22.2 (DO), LED23.3 (DI)
- new net: LED19.2 (DO), LED20.3 (DI)
- new net: LED23.2 (DO), LED24.3 (DI)

Commit message: add jlcpscb folder
Parts:
- F1: LCSC # (none) -> C883162
Changed lines of the file:
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@@
       (effects (font (size 1.27 1.27)) (justify left) hide)
+    )
+    (property "LCSC #" "C883162" (id 4) (at 269.24 137.16 0)
+      (effects (font (size 1.27 1.27)) hide)
     )
     (pin "1")

Commit message: added groundplate, update gitignore
Parts:
- LED1, LED10, LED11, LED12, LED13, LED14, LED15, LED16, LED17, LED18, LED19, LED2, LED20, LED21, LED22, LED23, LED24, LED25, LED26, LED27, LED28, LED29, LED3, LED30, LED4, LED5, LED6, LED7, LED8, LED9: footprint footprint:LED-SMD_4P-L5.0-W5.0-BL_XL-5050RGBC -> LED_SMD:LED_WS2812B_PLCC4_5.0x5.0mm_P3.2mm

Commit message: add open hardware logo and some text, resolved warnings
Parts:
- removed F1: BSMD1812-300-16V, footprint:F1812, symbol GLOWINGKITTYPARTS:BSMD1812-300-16V
- added F?: BSMD1812-300-16V, footprint:F1812, symbol GLOWINGKITTYPARTS:BSMD1812-300-16V
Connections:
- net +5V: now also F?.2
- net VBUS: now also F?.1
Changed lines of the file:
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@@
     (pin "4")
-  )
-  (symbol (lib_id "GLOWINGKITTYPARTS:BSMD1812-300-16V") (at 269.24 137.16 0) (unit 1)
-    (in_bom yes) (on_board yes) (fields_autoplaced)
-    (property "Reference" "F1" (id 0) (at 269.24 143.51 0))
-    (property "Value" "BSMD1812-300-16V" (id 1) (at 269.24 146.05 0))
-    (property "Footprint" "footprint:F1812" (id 2) (at 269.24 147.32 0)
-      (effects (font (size 1.27 1.27) italic) hide)
-    )
-    (property "Datasheet" "https://item.szlcsc.com/343302.html" (id 3) (at 266.954 137.033 0)
-      (effects (font (size 1.27 1.27)) (justify left) hide)
-    )
-    (property "LCSC #" "C883162" (id 4) (at 269.24 137.16 0)
-      (effects (font (size 1.27 1.27)) hide)
-    )
-    (pin "1")
-    (pin "2")
   )
   (symbol (lib_id "Device:C") (at 115.57 168.91 0) (unit 1)
@@
     (pin "1")
   )
+  (symbol (lib_id "GLOWINGKITTYPARTS:BSMD1812-300-16V") (at 269.24 137.16 0) (unit 1)
+    (in_bom yes) (on_board yes) (fields_autoplaced)
+    (property "Reference" "F?" (id 0) (at 269.24 143.51 0))
+    (property "Value" "BSMD1812-300-16V" (id 1) (at 269.24 146.05 0))
+    (property "Footprint" "footprint:F1812" (id 2) (at 269.24 147.32 0)
+      (effects (font (size 1.27 1.27) italic) hide)
+    )
+    (property "Datasheet" "https://item.szlcsc.com/343302.html" (id 3) (at 266.954 137.033 0)
+      (effects (font (size 1.27 1.27)) (justify left) hide)
+    )
+    (pin "1")
+    (pin "2")
+  )
   (symbol (lib_id "power:GND") (at 110.49 231.14 270) (unit 1)
     (in_bom yes) (on_board yes) (fields_autoplaced)
@@
       (reference "C39") (unit 1) (value "1nF") (footprint "Capacitor_SMD:C_0603_1608Metric_Pad1.08x0.95mm_HandSolder")
     )
-    (path "/551519e0-f194-4fea-aa92-4bfe8e6cee56"
-      (reference "F1") (unit 1) (value "BSMD1812-300-16V") (footprint "footprint:F1812")
+    (path "/abf2a1f7-98bd-4225-aa63-811aa466dc2c"
+      (reference "F?") (unit 1) (value "BSMD1812-300-16V") (footprint "footprint:F1812")
     )
     (path "/50c7f2f4-0373-4c85-ae8a-5b6178a8a88d"
